Commit message: removed static link

File: t42_gripper_description/urdf/hand_T42.xacro (robot description, xacro)
@@ -162,9 +162,4 @@
         </collision>
     </link>
-    <joint name="world_to_base" type="fixed">
-        <origin rpy="0 0 0" xyz="0 0 0" />
-        <parent link="world" />
-        <child link="base_link" />
-    </joint>
     <joint name="base_link_to_swivel_1" type="fixed">
         <origin rpy="0 0 0" xyz="0 0.000000 0.000000" />
