Commit message: Update controllers Add Rviz Change srdf to xacro

File: t42_gripper_description/urdf/t42.ros2_control.xacro (robot description, xacro)
@@ -16,5 +16,5 @@
         <command_interface name="position">
           <param name="min">0</param>
-          <param name="max">3</param>
+          <param name="max">1.57</param>
         </command_interface>
         <command_interface name="velocity">
@@ -44,5 +44,5 @@
         <command_interface name="position">
           <param name="min">0</param>
-          <param name="max">3</param>
+          <param name="max">1.57</param>
         </command_interface>
         <command_interface name="velocity">

File: t42_gripper_description/urdf/t42_hand_macro.xacro (robot description, xacro)
@@ -49,10 +49,10 @@
             izz="0.0"/>
         </inertial> -->
-        <!-- <collision>
-        <origin rpy="1.57 0 -1.57" xyz="0.06 0.017 0"/>
-        <geometry>
-            <mesh filename="package://t42_gripper_description/meshes/t42_base_link.STL"/>
-        </geometry>
-        </collision> -->
+        <collision>
+            <origin rpy="0 0 1.57" xyz="0.1 -0.035 -0.09"/>
+            <geometry>
+                <mesh filename="package://t42_gripper_description/meshes/actuator_block_t42.stl"/>
+            </geometry>
+        </collision>
     </link>
     <link name="swivel_1">
@@ -66,4 +66,10 @@
             </geometry>
         </visual>
+        <collision>
+            <origin rpy="0 1.57 1.57" xyz="-0.016510 ${swivel_distance} 0" />
+            <geometry>
+                <mesh filename="package://t42_gripper_description/meshes/swivel_t42.STL" scale="0.001 0.001 0.001" />
+            </geometry>
+        </collision>
     </link>
     <link name="finger_1_1">
@@ -122,4 +128,10 @@
             </geometry>
         </visual>
+        <collision>
+            <origin rpy="0 1.57 1.57" xyz="-0.016510 -${swivel_distance} 0" />
+            <geometry>
+                <mesh filename="package://t42_gripper_description/meshes/swivel_t42.STL" scale="0.001 0.001 0.001" />
+            </geometry>
+        </collision>
     </link>
     <link name="finger_2_1">
@@ -176,5 +188,5 @@
         <parent link="swivel_1" />
         <child link="finger_1_1" />
-        <limit effort="10000" lower="0.0" upper="3.0" velocity="2" />
+        <limit effort="10000" lower="0.0" upper="2" velocity="2" />
         <axis xyz="1 0 0" />
         <dynamics damping="${joint_damping_coefficient}" friction="${joint_friction_coefficient}" />
@@ -197,5 +209,5 @@
         <parent link="swivel_2" />
         <child link="finger_2_1" />
-        <limit effort="10000" lower="0.0" upper="3.0" velocity="2" />
+        <limit effort="10000" lower="0.0" upper="2" velocity="2" />
         <axis xyz="1 0 0" />
         <dynamics damping="${joint_damping_coefficient}" friction="${joint_friction_coefficient}" />
@@ -209,5 +221,5 @@
         <dynamics damping="${joint_damping_coefficient}" friction="${joint_friction_coefficient}" />
     </joint>
- <!-- Transmissions -->
+ <!-- Transmissions
   <transmission name="finger1_2_trans" type="SimpleTransmission">
       <type>transmission_interface/SimpleTransmission</type>
@@ -245,5 +257,5 @@
           <hardwareInterface>hardware_interface/EffortJointInterface</hardwareInterface>
       </joint>
-  </transmission>
+  </transmission> -->
 </xacro:macro>
 </robot>
