Commit message: working moveit control

File: t42_gripper_description/urdf/t42_hand_macro.xacro (robot description, xacro)
@@ -1,4 +1,10 @@
 <?xml version="1.0"?>
-<robot xmlns:xacro="http://www.ros.org/wiki/xacro" name="hand_T42_model">
+<robot xmlns:xacro="http://www.ros.org/wiki/xacro" >
+    <xacro:macro name="t42_hand" params="name:=hand_T42_model use_fake_hardware:=true">
+    <xacro:include filename="$(find t42_gripper_description)/urdf/t42.ros2_control.xacro" />
+    <!-- ros2 control instance -->
+    <xacro:tr42_ros2_control
+      name="TR42PositionHardwareInterface"
+      use_fake_hardware="$(arg use_fake_hardware)"/>
  	<xacro:macro name="base_color">
  		<color rgba="0.1 0.1 0.1 1"/>
@@ -25,8 +31,7 @@
     <xacro:property name="joint_damping_coefficient" value="7.0" />
     <xacro:property name="joint_friction_coefficient" value="0.0" />
-    <link name="world" />
-    <link name="base_link">
-        <visual>
-            <origin rpy="0 0 1.57" xyz="0.1 -0.035 -0.095"/>
+    <link name="t42_base_link">
+        <visual>
+            <origin rpy="0 0 1.57" xyz="0.1 -0.035 -0.09"/>
             <geometry>
                 <mesh filename="package://t42_gripper_description/meshes/actuator_block_t42.stl"/>
@@ -47,5 +52,5 @@
         <origin rpy="1.57 0 -1.57" xyz="0.06 0.017 0"/>
         <geometry>
-            <mesh filename="package://t42_gripper_description/meshes/base_link.STL"/>
+            <mesh filename="package://t42_gripper_description/meshes/t42_base_link.STL"/>
         </geometry>
         </collision> -->
@@ -162,7 +167,7 @@
         </collision>
     </link>
-    <joint name="base_link_to_swivel_1" type="fixed">
+    <joint name="t42_base_link_to_swivel_1" type="fixed">
         <origin rpy="0 0 0" xyz="0 0.000000 0.000000" />
-        <parent link="base_link" />
+        <parent link="t42_base_link" />
         <child link="swivel_1" />
     </joint>
@@ -183,7 +188,7 @@
         <dynamics damping="${joint_damping_coefficient}" friction="${joint_friction_coefficient}" />
     </joint>
-    <joint name="base_link_to_swivel_2" type="fixed">
+    <joint name="t42_base_link_to_swivel_2" type="fixed">
         <origin rpy="0 0 0" xyz="0 0.000000 0.000000" />
-        <parent link="base_link" />
+        <parent link="t42_base_link" />
         <child link="swivel_2" />
     </joint>
@@ -241,3 +246,4 @@
       </joint>
   </transmission>
+</xacro:macro>
 </robot>

Commit message: Add arduino controller file

File: t42_gripper_description/urdf/t42_hand_macro.xacro (robot description, xacro)
@@ -56,4 +56,54 @@
         </collision>
     </link>
+    <link name="arduino_controller">
+        <visual>
+            <origin xyz="0 0 0" rpy="0 0 0"/>
+            <geometry>
+                <mesh filename="package://t42_gripper_description/meshes/arduino_controller.stl"/>
+            </geometry>
+            <material name="black">
+                <color rgba="0.1 0.1 0.1 1"/>
+            </material>
+        </visual>
+        <!-- <inertial>
+            <origin xyz="0 0 0" rpy="0 0 0"/>
+            <mass value="0.1"/>
+            <inertia
+            ixx="0.0" ixy="0.0" ixz="0.0"
+            iyy="0.0" iyz="0.0"
+            izz="0.0"/>
+        </inertial> -->
+        <collision>
+            <origin xyz="0 0 0" rpy="0 0 0"/>
+            <geometry>
+                <mesh filename="package://t42_gripper_description/meshes/arduino_controller.stl"/>
+            </geometry>
+        </collision>
+    </link>
+    <link name="arduino_pc">
+        <visual>
+            <origin xyz="0 0 0" rpy="0 0 0"/>
+            <geometry>
+                <mesh filename="package://t42_gripper_description/meshes/arduino_pc.stl"/>
+            </geometry>
+            <material name="black">
+                <color rgba="0.1 0.1 0.1 1"/>
+            </material>
+        </visual>
+        <!-- <inertial>
+            <origin xyz="0 0 0" rpy="0 0 0"/>
+            <mass value="0.1"/>
+            <inertia
+            ixx="0.0" ixy="0.0" ixz="0.0"
+            iyy="0.0" iyz="0.0"
+            izz="0.0"/>
+        </inertial> -->
+        <collision>
+            <origin xyz="0 0 0" rpy="0 0 0"/>
+            <geometry>
+                <mesh filename="package://t42_gripper_description/meshes/arduino_pc.stl"/>
+            </geometry>
+        </collision>
+    </link>
     <link name="swivel_1">
         <visual>
@@ -183,4 +233,14 @@
         <parent link="t42_base_link" />
         <child link="swivel_1" />
+    </joint>
+    <joint name="t42_base_link_to_arduino_pc" type="fixed">
+        <origin rpy="1.57 0 1.57" xyz="0.02655 0.0 0.05153"/>
+        <parent link="t42_base_link" />
+        <child link="arduino_pc" />
+    </joint>
+    <joint name="t42_base_link_to_arduino_controller" type="fixed">
+        <origin rpy="1.57 0 1.57" xyz="0.02655 0.0 -0.059"/>
+        <parent link="t42_base_link" />
+        <child link="arduino_controller" />
     </joint>
     <joint name="swivel_1_to_finger_1_1" type="revolute">
